File: Hardware/Project.kicad_sch (KiCad schematic)
At the start: 10 parts, among them IC1 CD4017BE, IC2 NE555P, J1 Barrel_Jack_Switch, J2 Socket_CD4017BE, J3 Socket_NE555, U1 74AHC1G00

Commit message: library manager v1.1
Parts:
- removed C1: 10uF/25V, Capacitor_THT:CP_Radial_D4.0mm_P2.00mm, symbol Device:C_Polarized_Small
- removed H1: MountingHole, MountingHole:MountingHole_3.2mm_M3, symbol Mechanical:MountingHole
- removed IC1: CD4017BE, ProjectFootprints:CD4017BE, symbol ProjectSymbols:CD4017BE
- removed IC2: NE555P, ProjectFootprints:NE555P, symbol ProjectSymbols:NE555P
- removed J1: Barrel_Jack_Switch, Connector_BarrelJack:BarrelJack_Horizontal, symbol Connector:Barrel_Jack_Switch
- removed J2: Socket_CD4017BE, symbol Connector_Generic:Conn_02x08_Counter_Clockwise
- removed J3: Socket_NE555, symbol Connector_Generic:Conn_02x04_Counter_Clockwise
- removed R25: 10k, Resistor_THT:R_Axial_DIN0204_L3.6mm_D1.6mm_P7.62mm_Horizontal, symbol Device:R_Small
- removed RV1: 10k_Poti, Potentiometer_THT:Potentiometer_Runtron_RM-065_Vertical, symbol Device:R_Potentiometer_Small
- removed U1: 74AHC1G00, symbol 74xGxx:74AHC1G00
Connections:
- no-connect marks 10 -> 0
Other:
- removed sheet LED_BLUE
- removed sheet LED_GREEN
- removed sheet LED_RED
