File: Hardware/Project.kicad_sch (KiCad schematic)
At the start: 0 parts

Commit message: mouser auto fix
Parts:
- added H1, H2, H3, H4: MountingHole, MountingHole:MountingHole_2.7mm_M2.5, symbol Mechanical:MountingHole
Other:
- added sheet ADS1015 (ads1015.kicad_sch)
- added sheet ELRS_Transceiver (ELRS_transceiver.kicad_sch)
- added sheet ESP32 (esp32.kicad_sch)
- added sheet Joysticks (joysticks.kicad_sch)
- added sheet SD-Card (sd-card.kicad_sch)
- added sheet Supply (supply.kicad_sch)
- added sheet Tactile_Switches (tactile_switches.kicad_sch)
